File: mainboard/main.kicad_pcb (KiCad board)
At the start: 2 copper layers, 13 parts, among them J1 Conn_01x02, J2 Conn_01x15_Female, J3 Conn_01x11_Female, J4 Conn_01x15_Female, J5 Conn_01x04_Female, J6 Conn_01x06_Female, SW1 SW_MEC_5G, U1 ATtiny45-20PU

Commit message: Add files via upload
Parts:
- removed SW1: SW_MEC_5G, Button_Switch_THT:SW_NKK_GW12LJP
- added J7: Conn_01x04_Female, Connector_PinSocket_2.54mm:PinSocket_1x04_P2.54mm_Vertical, F.Cu at (255.9, 56.0)
- added J8: Conn_02x03_Counter_Clockwise, Connector_PinSocket_2.54mm:PinSocket_2x03_P2.54mm_Vertical, F.Cu at (172.7, 99.1)
- H1, H2, H3, H4: footprint MountingHole:MountingHole_3mm -> MountingHole:MountingHole_3.2mm_M3_DIN965_Pad
- J6: value Conn_01x06_Female -> Conn_01x04_Female; footprint Connector_PinSocket_2.54mm:PinSocket_1x06_P2.54mm_Vertical -> Connector_PinSocket_2.54mm:PinSocket_1x04_P2.54mm_Vertical
- moved H3 8.89 mm to (250.2, 45.7)
- moved H4 8.89 mm to (250.2, 106.7)
- moved J6 7.49 mm to (251.3, 56.0), turned to 0 degrees
Connections:
- J6 pad 1: (no net) -> Net-(J6-Pad1)
- J6 pad 2: (no net) -> Net-(J6-Pad2)
- J6 pad 3: (no net) -> Net-(J6-Pad3)
- J6 pad 4: (no net) -> Net-(J6-Pad4)
Routing:
- net Net-(J6-Pad4): track 0.00 -> 4.60 mm
- net Net-(J6-Pad3): track 0.00 -> 4.60 mm
- net Net-(J6-Pad2): track 0.00 -> 4.60 mm
- net Net-(J6-Pad1): track 0.00 -> 4.60 mm

Commit message: Add files via upload
Parts:
- moved J1 7.73 mm to (170.2, 69.8)
Routing:
- net (no net): track 62.8 -> 54.6 mm
- net Net-(J1-Pad1): track 30.5 -> 24.1 mm
Changed lines of the file:
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@@
     (thickness 1.6)
     (drawings 2)
-    (tracks 85)
+    (tracks 83)
     (zones 0)
     (modules 14)
@@
   )
   (setup
-    (last_trace_width 0.25)
+    (last_trace_width 2)
     (user_trace_width 1.2)
     (user_trace_width 2)
@@
     (uvia_drill 0.1)
     (add_net CLK)
-    (add_net D0)
     (add_net D1)
     (add_net D2)
@@
     (add_net MOSI)
     (add_net "Net-(J1-Pad1)")
-    (add_net "Net-(J2-Pad1)")
-    (add_net "Net-(J2-Pad10)")
     (add_net "Net-(J2-Pad11)")
-    (add_net "Net-(J2-Pad12)")
-    (add_net "Net-(J2-Pad13)")
     (add_net "Net-(J2-Pad14)")
-    (add_net "Net-(J2-Pad2)")
-    (add_net "Net-(J2-Pad3)")
-    (add_net "Net-(J2-Pad4)")
-    (add_net "Net-(J2-Pad5)")
-    (add_net "Net-(J2-Pad6)")
-    (add_net "Net-(J2-Pad7)")
-    (add_net "Net-(J2-Pad8)")
-    (add_net "Net-(J2-Pad9)")
     (add_net "Net-(J3-Pad4)")
-    (add_net "Net-(J4-Pad14)")
-    (add_net "Net-(J4-Pad6)")
     (add_net "Net-(J4-Pad7)")
     (add_net "Net-(J6-Pad1)")
@@
     (add_net "Net-(J6-Pad3)")
     (add_net "Net-(J6-Pad4)")
-    (add_net "Net-(J8-Pad1)")
-    (add_net "Net-(J8-Pad2)")
-    (add_net "Net-(J8-Pad3)")
-    (add_net "Net-(J8-Pad4)")
-    (add_net "Net-(J8-Pad5)")
-    (add_net "Net-(J8-Pad6)")
-    (add_net "Net-(U1-Pad1)")
-    (add_net "Net-(U1-Pad6)")
     (add_net RX)
-    (add_net TX)
     (add_net Up)
     (add_net VI)
@@
   )
   (module Connector_Wire:SolderWirePad_1x02_P5.08mm_Drill1.5mm (layer F.Cu)
-    (at 168.91 62.23)
+    (at 170.18 69.85)
     (descr "Wire solder connection")
     (tags connector)
@@
   (segment (start 170.18 86.36) (end 170.18 99.06) (width 2) (layer B.Cu) (net 0))
   (segment (start 170.1 86.28) (end 170.18 86.36) (width 2) (layer B.Cu) (net 0))
-  (segment (start 175.26 64.460118) (end 175.26 99.06) (width 2) (layer B.Cu) (net 0))
-  (segment (start 173.99 63.190118) (end 175.26 64.460118) (width 2) (layer B.Cu) (net 0))
-  (segment (start 173.99 62.23) (end 173.99 63.190118) (width 2) (layer B.Cu) (net 0))
-  (segment (start 157.48 81.28) (end 157.48 62.23) (width 2) (layer B.Cu) (net 1))
-  (segment (start 157.48 62.23) (end 168.91 62.23) (width 2) (layer B.Cu) (net 1))
+  (segment (start 175.26 69.85) (end 175.26 99.06) (width 2) (layer B.Cu) (net 0))
+  (segment (start 157.48 81.28) (end 170.18 81.28) (width 2) (layer B.Cu) (net 1))
+  (segment (start 170.18 81.28) (end 170.18 69.85) (width 2) (layer B.Cu) (net 1))
   (segment (start 186.88 91.48) (end 186.88 86.55) (width 1.2) (layer B.Cu) (net 2))
   (segment (start 187.07 86.36) (end 193.04 86.36) (width 1.2) (layer B.Cu) (net 2))
@@
   (segment (start 251.46 58.42) (end 256.06 58.42) (width 1.2) (layer B.Cu) (net 21))
   (segment (start 251.333 56.007) (end 255.933 56.007) (width 1.2) (layer B.Cu) (net 22))
+  (zone (net 0) (net_name "") (layer B.Cu) (hatch full 0.508)
+    (connect_pads (clearance 0.508))
+    (min_thickness 0.254)
+    (keepout (tracks allowed) (vias allowed) (copperpour not_allowed))
+    (fill (arc_segments 32) (thermal_gap 0.508) (thermal_bridge_width 0.508))
+    (polygon
+      (pts
+        (xy 154.94 66.04) (xy 154.94 100.33) (xy 154.94 106.68) (xy 182.88 106.68) (xy 182.88 66.04)
+      )
+    )
+  )
 )

Commit message: Add files via upload
Parts:
- added REF**: PinHeader_1x02_P2.54mm_Vertical, Connector_PinHeader_2.54mm:PinHeader_1x02_P2.54mm_Vertical, F.Cu at (230.6, 78.7)
- moved J7 3.15 mm to (259.1, 55.9)
- moved J6 0.18 mm to (251.5, 55.9)
Routing:
- net (no net): track 54.6 -> 64.3 mm
- net Net-(J6-Pad4): track 4.60 -> 7.62 mm
- net Net-(J6-Pad3): track 4.60 -> 7.62 mm
- net Net-(J6-Pad2): track 4.60 -> 7.62 mm
- net Net-(J6-Pad1): track 4.60 -> 7.62 mm
Changed lines of the file:
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@@
     (thickness 1.6)
     (drawings 2)
-    (tracks 83)
+    (tracks 84)
     (zones 0)
-    (modules 14)
+    (modules 15)
     (nets 23)
   )
@@
   )
   (setup
-    (last_trace_width 2)
+    (last_trace_width 1.2)
     (user_trace_width 1.2)
     (user_trace_width 2)
@@
     (add_net VI)
   )
+  (module Connector_PinSocket_2.54mm:PinSocket_1x04_P2.54mm_Vertical (layer F.Cu)
+    (at 251.46 55.88)
+    (descr "Through hole straight socket strip, 1x04, 2.54mm pitch, single row (from Kicad 4.0.7), script generated")
+    (tags "Through hole socket strip THT 1x04 2.54mm single row")
+    (fp_text reference J6 (at 0 -2.77) (layer F.SilkS)
+      (effects (font (size 1 1) (thickness 0.15)))
+    )
+    (fp_text value Conn_01x04_Female (at 0 10.39) (layer F.Fab)
+      (effects (font (size 1 1) (thickness 0.15)))
+    )
+    (fp_text user %R (at 0 3.81 90) (layer F.Fab)
+      (effects (font (size 1 1) (thickness 0.15)))
+    )
+    (fp_line (start -1.8 9.4) (end -1.8 -1.8) (layer F.CrtYd) (width 0.05))
+    (fp_line (start 1.75 9.4) (end -1.8 9.4) (layer F.CrtYd) (width 0.05))
+    (fp_line (start 1.75 -1.8) (end 1.75 9.4) (layer F.CrtYd) (width 0.05))
+    (fp_line (start -1.8 -1.8) (end 1.75 -1.8) (layer F.CrtYd) (width 0.05))
+    (fp_line (start 0 -1.33) (end 1.33 -1.33) (layer F.SilkS) (width 0.12))
+    (fp_line (start 1.33 -1.33) (end 1.33 0) (layer F.SilkS) (width 0.12))
+    (fp_line (start 1.33 1.27) (end 1.33 8.95) (layer F.SilkS) (width 0.12))
+    (fp_line (start -1.33 8.95) (end 1.33 8.95) (layer F.SilkS) (width 0.12))
+    (fp_line (start -1.33 1.27) (end -1.33 8.95) (layer F.SilkS) (width 0.12))
+    (fp_line (start -1.33 1.27) (end 1.33 1.27) (layer F.SilkS) (width 0.12))
+    (fp_line (start -1.27 8.89) (end -1.27 -1.27) (layer F.Fab) (width 0.1))
+    (fp_line (start 1.27 8.89) (end -1.27 8.89) (layer F.Fab) (width 0.1))
+    (fp_line (start 1.27 -0.635) (end 1.27 8.89) (layer F.Fab) (width 0.1))
+    (fp_line (start 0.635 -1.27) (end 1.27 -0.635) (layer F.Fab) (width 0.1))
+    (fp_line (start -1.27 -1.27) (end 0.635 -1.27) (layer F.Fab) (width 0.1))
+    (fp_line (start -1.33 -3.81) (end 1.33 -3.81) (layer F.SilkS) (width 0.12))
+    (fp_text user %R (at 0 -1.27 90) (layer F.Fab)
+      (effects (font (size 1 1) (thickness 0.15)))
+    )
+    (pad 4 thru_hole roundrect (at 0 7.62) (size 2.6 2) (drill 1) (layers *.Cu *.Mask) (roundrect_rratio 0.25)
+      (net 19 "Net-(J6-Pad4)"))
+    (pad 3 thru_hole roundrect (at 0 5.08) (size 2.6 2) (drill 1) (layers *.Cu *.Mask) (roundrect_rratio 0.25)
+      (net 20 "Net-(J6-Pad3)"))
+    (pad 2 thru_hole roundrect (at 0 2.54) (size 2.6 2) (drill 1) (layers *.Cu *.Mask) (roundrect_rratio 0.25)
+      (net 21 "Net-(J6-Pad2)"))
+    (pad 1 thru_hole roundrect (at 0 0) (size 2.6 2) (drill 1) (layers *.Cu *.Mask) (roundrect_rratio 0.25)
+      (net 22 "Net-(J6-Pad1)"))
+    (pad 2 thru_hole roundrect (at 0 -2.54) (size 2.6 2) (drill 1) (layers *.Cu *.Mask) (roundrect_rratio 0.25)
+      (net 21 "Net-(J6-Pad2)"))
+    (pad 1 thru_hole roundrect (at 0 -5.08) (size 2.6 2) (drill 1) (layers *.Cu *.Mask) (roundrect_rratio 0.25)
+      (net 22 "Net-(J6-Pad1)"))
+    (model ${KISYS3DMOD}/Connector_PinSocket_2.54mm.3dshapes/PinSocket_1x04_P2.54mm_Vertical.wrl
+      (at (xyz 0 0 0))
+      (scale (xyz 1 1 1))
+      (rotate (xyz 0 0 0))
+    )
+  )
+  (module Connector_PinHeader_2.54mm:PinHeader_1x02_P2.54mm_Vertical (layer F.Cu)
+    (at 230.632 78.74)
+    (descr "Through hole straight pin header, 1x02, 2.54mm pitch, single row")
+    (tags "Through hole pin header THT 1x02 2.54mm single row")
+    (fp_text reference REF** (at 0 -2.33) (layer F.SilkS)
+      (effects (font (size 1 1) (thickness 0.15)))
+    )
+    (fp_text value PinHeader_1x02_P2.54mm_Vertical (at 0 4.87) (layer F.Fab)
+      (effects (font (size 1 1) (thickness 0.15)))
+    )
+    (fp_text user %R (at 0 1.27 90) (layer F.Fab)
+      (effects (font (size 1 1) (thickness 0.15)))
+    )
+    (fp_line (start 1.8 -1.8) (end -1.8 -1.8) (layer F.CrtYd) (width 0.05))
+    (fp_line (start 1.8 4.35) (end 1.8 -1.8) (layer F.CrtYd) (width 0.05))
+    (fp_line (start -1.8 4.35) (end 1.8 4.35) (layer F.CrtYd) (width 0.05))
+    (fp_line (start -1.8 -1.8) (end -1.8 4.35) (layer F.CrtYd) (width 0.05))
+    (fp_line (start -1.33 -1.33) (end 0 -1.33) (layer F.SilkS) (width 0.12))
+    (fp_line (start -1.33 0) (end -1.33 -1.33) (layer F.SilkS) (width 0.12))
+    (fp_line (start -1.33 1.27) (end 1.33 1.27) (layer F.SilkS) (width 0.12))
+    (fp_line (start 1.33 1.27) (end 1.33 3.87) (layer F.SilkS) (width 0.12))
+    (fp_line (start -1.33 1.27) (end -1.33 3.87) (layer F.SilkS) (width 0.12))
+    (fp_line (start -1.33 3.87) (end 1.33 3.87) (layer F.SilkS) (width 0.12))
+    (fp_line (start -1.27 -0.635) (end -0.635 -1.27) (layer F.Fab) (width 0.1))
+    (fp_line (start -1.27 3.81) (end -1.27 -0.635) (layer F.Fab) (width 0.1))
+    (fp_line (start 1.27 3.81) (end -1.27 3.81) (layer F.Fab) (width 0.1))
+    (fp_line (start 1.27 -1.27) (end 1.27 3.81) (layer F.Fab) (width 0.1))
+    (fp_line (start -0.635 -1.27) (end 1.27 -1.27) (layer F.Fab) (width 0.1))
+    (pad 2 thru_hole roundrect (at 0 2.54) (size 2.6 2) (drill 1) (layers *.Cu *.Mask) (roundrect_rratio 0.25))
+    (pad 1 thru_hole roundrect (at 0 0) (size 2.6 2) (drill 1) (layers *.Cu *.Mask) (roundrect_rratio 0.25))
+    (model ${KISYS3DMOD}/Connector_PinHeader_2.54mm.3dshapes/PinHeader_1x02_P2.54mm_Vertical.wrl
+      (at (xyz 0 0 0))
+      (scale (xyz 1 1 1))
+      (rotate (xyz 0 0 0))
+    )
+  )
   (module Connector_PinSocket_2.54mm:PinSocket_2x03_P2.54mm_Vertical (layer F.Cu)
     (at 172.72 99.06 90)
@@
   )
   (module Connector_PinSocket_2.54mm:PinSocket_1x04_P2.54mm_Vertical (layer F.Cu)
-    (at 251.333 56.007)
-    (descr "Through hole straight socket strip, 1x04, 2.54mm pitch, single row (from Kicad 4.0.7), script generated")
-    (tags "Through hole socket strip THT 1x04 2.54mm single row")
-    (fp_text reference J6 (at 0 -2.77) (layer F.SilkS)
-      (effects (font (size 1 1) (thickness 0.15)))
-    )
-    (fp_text value Conn_01x04_Female (at 0 10.39) (layer F.Fab)
-      (effects (font (size 1 1) (thickness 0.15)))
-    )
-    (fp_text user %R (at 0 3.81 90) (layer F.Fab)
-      (effects (font (size 1 1) (thickness 0.15)))
-    )
-    (fp_line (start -1.8 9.4) (end -1.8 -1.8) (layer F.CrtYd) (width 0.05))
-    (fp_line (start 1.75 9.4) (end -1.8 9.4) (layer F.CrtYd) (width 0.05))
-    (fp_line (start 1.75 -1.8) (end 1.75 9.4) (layer F.CrtYd) (width 0.05))
-    (fp_line (start -1.8 -1.8) (end 1.75 -1.8) (layer F.CrtYd) (width 0.05))
-    (fp_line (start 0 -1.33) (end 1.33 -1.33) (layer F.SilkS) (width 0.12))
-    (fp_line (start 1.33 -1.33) (end 1.33 0) (layer F.SilkS) (width 0.12))
-    (fp_line (start 1.33 1.27) (end 1.33 8.95) (layer F.SilkS) (width 0.12))
-    (fp_line (start -1.33 8.95) (end 1.33 8.95) (layer F.SilkS) (width 0.12))
-    (fp_line (start -1.33 1.27) (end -1.33 8.95) (layer F.SilkS) (width 0.12))
-    (fp_line (start -1.33 1.27) (end 1.33 1.27) (layer F.SilkS) (width 0.12))
-    (fp_line (start -1.27 8.89) (end -1.27 -1.27) (layer F.Fab) (width 0.1))
-    (fp_line (start 1.27 8.89) (end -1.27 8.89) (layer F.Fab) (width 0.1))
-    (fp_line (start 1.27 -0.635) (end 1.27 8.89) (layer F.Fab) (width 0.1))
-    (fp_line (start 0.635 -1.27) (end 1.27 -0.635) (layer F.Fab) (width 0.1))
-    (fp_line (start -1.27 -1.27) (end 0.635 -1.27) (layer F.Fab) (width 0.1))
-    (pad 4 thru_hole roundrect (at 0 7.62) (size 2.6 2) (drill 1) (layers *.Cu *.Mask) (roundrect_rratio 0.25)
-      (net 19 "Net-(J6-Pad4)"))
-    (pad 3 thru_hole roundrect (at 0 5.08) (size 2.6 2) (drill 1) (layers *.Cu *.Mask) (roundrect_rratio 0.25)
-      (net 20 "Net-(J6-Pad3)"))
-    (pad 2 thru_hole roundrect (at 0 2.54) (size 2.6 2) (drill 1) (layers *.Cu *.Mask) (roundrect_rratio 0.25)
-      (net 21 "Net-(J6-Pad2)"))
-    (pad 1 thru_hole roundrect (at 0 0) (size 2.6 2) (drill 1) (layers *.Cu *.Mask) (roundrect_rratio 0.25)
-      (net 22 "Net-(J6-Pad1)"))
-    (model ${KISYS3DMOD}/Connector_PinSocket_2.54mm.3dshapes/PinSocket_1x04_P2.54mm_Vertical.wrl
-      (at (xyz 0 0 0))
-      (scale (xyz 1 1 1))
-      (rotate (xyz 0 0 0))
-    )
-  )
-  (module Connector_PinSocket_2.54mm:PinSocket_1x04_P2.54mm_Vertical (layer F.Cu)
-    (at 255.933 56.007)
+    (at 259.08 55.88)
     (descr "Through hole straight socket strip, 1x04, 2.54mm pitch, single row (from Kicad 4.0.7), script generated")
     (tags "Through hole socket strip THT 1x04 2.54mm single row")
@@
   (segment (start 170.1 86.28) (end 170.18 86.36) (width 2) (layer B.Cu) (net 0))
   (segment (start 175.26 69.85) (end 175.26 99.06) (width 2) (layer B.Cu) (net 0))
+  (segment (start 220.98 81.28) (end 230.632 81.28) (width 1.2) (layer B.Cu) (net 0))
   (segment (start 157.48 81.28) (end 170.18 81.28) (width 2) (layer B.Cu) (net 1))
   (segment (start 170.18 81.28) (end 170.18 69.85) (width 2) (layer B.Cu) (net 1))
@@
   (segment (start 231.14 58.42) (end 220.98 58.42) (width 1.2) (layer B.Cu) (net 17))
   (segment (start 231.14 55.88) (end 220.98 55.88) (width 1.2) (layer B.Cu) (net 18))
-  (segment (start 251.333 63.627) (end 255.933 63.627) (width 1.2) (layer B.Cu) (net 19))
-  (segment (start 251.333 60.96) (end 255.933 60.96) (width 1.2) (layer B.Cu) (net 20))
-  (segment (start 251.46 58.42) (end 256.06 58.42) (width 1.2) (layer B.Cu) (net 21))
-  (segment (start 251.333 56.007) (end 255.933 56.007) (width 1.2) (layer B.Cu) (net 22))
+  (segment (start 251.46 63.5) (end 259.08 63.5) (width 1.2) (layer B.Cu) (net 19))
+  (segment (start 251.46 60.96) (end 259.08 60.96) (width 1.2) (layer B.Cu) (net 20))
+  (segment (start 251.46 58.42) (end 259.08 58.42) (width 1.2) (layer B.Cu) (net 21))
+  (segment (start 251.46 55.88) (end 259.08 55.88) (width 1.2) (layer B.Cu) (net 22))
   (zone (net 0) (net_name "") (layer B.Cu) (hatch full 0.508)
     (connect_pads (clearance 0.508))
