File: lcd board/lcd board.kicad_pcb (KiCad board)
At the start: 2 copper layers, 12 parts, among them J1 Conn_01x11, SW1 SW_Push, SW2 SW_Push, SW3 SW_Push, U1 CR2013-MI2120

Commit message: Add files via upload
Parts:
- moved J1 25.4 mm to (119.4, 10.2), turned to 90 degrees
Connections:
- J1 pad 10: GND -> Net-(J1-Pad10)
- J1 pad 2: Net-(J1-Pad2) -> GND
- R1 pad 1: Net-(J1-Pad3) -> Net-(J1-Pad9)
- R2 pad 1: Net-(J1-Pad2) -> Net-(J1-Pad10)
- R3 pad 1: Net-(J1-Pad1) -> Net-(J1-Pad11)
- SW1 pad 1: Net-(J1-Pad4) -> Net-(J1-Pad8)
- SW1 pad 2: Net-(J1-Pad3) -> Net-(J1-Pad9)
- SW2 pad 1: Net-(J1-Pad4) -> Net-(J1-Pad8)
- SW2 pad 2: Net-(J1-Pad2) -> Net-(J1-Pad10)
- SW3 pad 1: Net-(J1-Pad4) -> Net-(J1-Pad8)
- SW3 pad 2: Net-(J1-Pad1) -> Net-(J1-Pad11)
- U1 pad 1: Net-(J1-Pad4) -> Net-(J1-Pad8)
- U1 pad 10: Net-(J1-Pad11) -> Net-(J1-Pad1)
- U1 pad 11: Net-(J1-Pad7) -> Net-(J1-Pad5)
- U1 pad 12: Net-(J1-Pad5) -> Net-(J1-Pad7)
- U1 pad 3: Net-(J1-Pad9) -> Net-(J1-Pad3)
- U1 pad 4: Net-(J1-Pad4) -> Net-(J1-Pad8)
- U1 pad 5: Net-(J1-Pad8) -> Net-(J1-Pad4)
- U1 pad 6: Net-(J1-Pad7) -> Net-(J1-Pad5)
- U1 pad 8: Net-(J1-Pad4) -> Net-(J1-Pad8)
- U1 pad 9: Net-(J1-Pad5) -> Net-(J1-Pad7)
Routing:
- net Net-(J1-Pad2): track 77.0 -> 0.00 mm
- net Net-(J1-Pad10): track 0.00 -> 77.0 mm
- net Net-(J1-Pad8): track 58.4 -> 111.2 mm
- net Net-(J1-Pad4): track 111.2 -> 58.4 mm
- net Net-(J1-Pad11): track 58.4 -> 94.6 mm
- net Net-(J1-Pad1): track 94.6 -> 58.4 mm
- net Net-(J1-Pad9): track 66.0 -> 58.1 mm
- net Net-(J1-Pad3): track 58.1 -> 66.0 mm
- net Net-(J1-Pad7): track 124.5 -> 126.6 mm
- net Net-(J1-Pad5): track 126.6 -> 124.5 mm
